File: KiCad projecten/Moederbord/Moederbord.kicad_pcb (KiCad board)
At the start: 2 copper layers, 150 x 150 mm, 30 parts, among them J13 Conn_01x06_Male, J14 Conn_01x06_Male, J15 Conn_01x06_Male, J16 Conn_01x06_Male, J17 Conn_01x06_Male, J18 Conn_01x06_Male, J19 Conn_01x06_Male, J20 Conn_01x06_Male, J21 Conn_01x06_Male, J22 Conn_01x06_Male, J23 Conn_01x06_Male, J24 Conn_01x06_Male, J25 Conn_01x06_Male, J26 Conn_01x06_Male, J27 Conn_01x06_Male, J28 Conn_01x06_Male, J29 Conn_01x06_Male, J30 Conn_01x06_Male, J31 Conn_01x06_Male, J32 Conn_01x06_Male, J33 Conn_01x06_Male, J34 Conn_01x06_Male, J35 Conn_01x06_Male, J36 Conn_01x06_Male, J37 Conn_01x06_Male, J7 Conn_01x15_Female, J8 Conn_01x15_Female, U1 74166, U2 74166, U3 74166

Commit message: Update na overleg
Parts:
- removed the J19 at (31.5, 68.5)
- removed the J7 at (85.0, 52.4)
- added J1: I2S_DAC, Socket_Strips:Socket_Strip_Straight_1x06_Pitch2.54mm, F.Cu at (127.0, 171.0)
- added J12: Conn_01x06_Male, Moederbord:IDC_Header_Straight_6pins, F.Cu at (31.5, 68.5)
- added J2: RFID_reader, Socket_Strips:Socket_Strip_Straight_1x08_Pitch2.54mm, F.Cu at (59.0, 171.0)
- added J3: ESP32_left, Socket_Strips:Socket_Strip_Straight_1x15_Pitch2.54mm, F.Cu at (85.0, 52.4)
- added REF**: MountingHole_3.2mm_M3_ISO14580, Mounting_Holes:MountingHole_3.2mm_M3_ISO14580, F.Cu at (169.0, 173.0)
- added REF**: MountingHole_3.2mm_M3_ISO14580, Mounting_Holes:MountingHole_3.2mm_M3_ISO14580, F.Cu at (27.0, 173.0)
- added REF**: MountingHole_3.2mm_M3_ISO14580, Mounting_Holes:MountingHole_3.2mm_M3_ISO14580, F.Cu at (27.0, 32.0)
- added REF**: MountingHole_3.2mm_M3_ISO14580, Mounting_Holes:MountingHole_3.2mm_M3_ISO14580, F.Cu at (169.0, 33.0)
- J4: renamed from J8; value Conn_01x15_Female -> ESP32_right; footprint Pin_Headers:Pin_Header_Straight_1x15_Pitch2.54mm -> Socket_Strips:Socket_Strip_Straight_1x15_Pitch2.54mm
- moved J14 4.00 mm to (35.5, 34.5)
- moved J15 4.00 mm to (52.5, 34.5)
- moved J16 4.00 mm to (69.5, 34.5)
- moved J17 4.00 mm to (86.5, 34.5)
- moved J18 4.00 mm to (103.9, 34.5)
- moved J19 4.00 mm to (121.0, 34.5)
- moved J20 4.00 mm to (138.0, 34.5)
- moved J21 4.00 mm to (155.0, 34.0)
- renumbered J17 to J10, J18 to J11, J20 to J13, J21 to J14, J22 to J15, J23 to J16, J24 to J17, J25 to J18, J26 to J19, J27 to J20, J28 to J21, J29 to J22, J30 to J23, J31 to J24, J32 to J25, J33 to J26, J34 to J27, J35 to J28, J36 to J29, J37 to J5, J13 to J6, J14 to J7, J15 to J8, J16 to J9
Connections:
- J29 pad 3: Net-(J36-Pad3) -> (no net)
- J5 pad 2: Net-(J36-Pad3) -> (no net)
- J5 pad 3: (no net) -> Net-(J5-Pad3)
- J6 pad 2: (no net) -> Net-(J5-Pad3)
- U1 pad 13: (no net) -> Net-(U1-Pad13)
- U2 pad 1: (no net) -> Net-(U1-Pad13)
- U2 pad 13: (no net) -> Net-(U2-Pad13)
- U3 pad 1: (no net) -> Net-(U2-Pad13)

Commit message: Update moederbord
Parts:
- removed the REF** at (169.0, 173.0)
- removed the REF** at (27.0, 173.0)
- removed the REF** at (27.0, 32.0)
- removed the REF** at (169.0, 33.0)
- added J30: Conn_01x06_Male, Moederbord:IDC_Header_Straight_6pins, F.Cu at (85.8, 100.5)
- added J31: Conn_01x06_Male, Moederbord:IDC_Header_Straight_6pins, F.Cu at (104.5, 100.5)
- added J32: Conn_01x06_Male, Moederbord:IDC_Header_Straight_6pins, F.Cu at (123.2, 100.5)
- added J33: Conn_01x06_Male, Moederbord:IDC_Header_Straight_6pins, F.Cu at (141.9, 100.5)
- added J34: Conn_01x06_Male, Moederbord:IDC_Header_Straight_6pins, F.Cu at (161.0, 101.0)
- added J35: Conn_01x06_Male, Moederbord:IDC_Header_Straight_6pins, F.Cu at (30.0, 159.0)
- added J36: Conn_01x06_Male, Moederbord:IDC_Header_Straight_6pins, F.Cu at (48.7, 159.0)
- added J37: Conn_01x06_Male, Moederbord:IDC_Header_Straight_6pins, F.Cu at (67.4, 159.0)
- added J38: Conn_01x06_Male, Moederbord:IDC_Header_Straight_6pins, F.Cu at (86.1, 159.0)
- added J39: Conn_01x06_Male, Moederbord:IDC_Header_Straight_6pins, F.Cu at (104.8, 159.0)
- added J40: Conn_01x06_Male, Moederbord:IDC_Header_Straight_6pins, F.Cu at (123.5, 159.0)
- added J41: Conn_01x06_Male, Moederbord:IDC_Header_Straight_6pins, F.Cu at (142.2, 159.0)
- added J42: Conn_01x06_Male, Moederbord:IDC_Header_Straight_6pins, F.Cu at (160.9, 159.0)
- added J43: Conn_02x01, Wire_Connections_Bridges:WireConnection_1.00mmDrill, F.Cu at (67.8, 209.0)
- added J44: Conn_02x01, Wire_Connections_Bridges:WireConnection_1.00mmDrill, F.Cu at (67.8, 212.0)
- added J45: Conn_02x01, Wire_Connections_Bridges:WireConnection_1.00mmDrill, F.Cu at (67.8, 215.0)
- added J46: Conn_02x01, Wire_Connections_Bridges:WireConnection_1.00mmDrill, F.Cu at (68.0, 218.0)
- added J47: Conn_02x01, Wire_Connections_Bridges:WireConnection_1.00mmDrill, F.Cu at (109.2, 222.0)
- added J48: Conn_02x01, Wire_Connections_Bridges:WireConnection_1.00mmDrill, F.Cu at (109.0, 219.0)
- added J49: Conn_02x01, Wire_Connections_Bridges:WireConnection_1.00mmDrill, F.Cu at (109.2, 217.0)
- added J50: Conn_02x01, Wire_Connections_Bridges:WireConnection_1.00mmDrill, F.Cu at (109.0, 212.0)
- added J51: Conn_02x01, Wire_Connections_Bridges:WireConnection_1.00mmDrill, F.Cu at (67.8, 232.0)
- added J52: Conn_02x01, Wire_Connections_Bridges:WireConnection_1.00mmDrill, F.Cu at (67.8, 235.0)
- added J53: Conn_02x01, Wire_Connections_Bridges:WireConnection_1.00mmDrill, F.Cu at (67.8, 238.0)
- added J54: Conn_02x01, Wire_Connections_Bridges:WireConnection_1.00mmDrill, F.Cu at (67.8, 241.0)
- added J55: Conn_02x01, Wire_Connections_Bridges:WireConnection_1.00mmDrill, F.Cu at (109.0, 246.0)
- added J56: Conn_02x01, Wire_Connections_Bridges:WireConnection_1.00mmDrill, F.Cu at (109.2, 243.0)
- added J57: Conn_02x01, Wire_Connections_Bridges:WireConnection_1.00mmDrill, F.Cu at (109.2, 240.0)
- added J58: Conn_02x01, Wire_Connections_Bridges:WireConnection_1.00mmDrill, F.Cu at (109.2, 236.0)
- added J59: Conn_02x01, Wire_Connections_Bridges:WireConnection_1.00mmDrill, F.Cu at (68.0, 256.0)
- added J60: Conn_02x01, Wire_Connections_Bridges:WireConnection_1.00mmDrill, F.Cu at (67.8, 259.0)
- added J61: Conn_02x01, Wire_Connections_Bridges:WireConnection_1.00mmDrill, F.Cu at (68.0, 262.0)
- added J62: Conn_02x01, Wire_Connections_Bridges:WireConnection_1.00mmDrill, F.Cu at (67.8, 265.0)
- added J63: Conn_02x01, Wire_Connections_Bridges:WireConnection_1.00mmDrill, F.Cu at (109.2, 270.0)
- added J64: Conn_02x01, Wire_Connections_Bridges:WireConnection_1.00mmDrill, F.Cu at (109.2, 267.0)
- added J65: Conn_02x01, Wire_Connections_Bridges:WireConnection_1.00mmDrill, F.Cu at (109.2, 264.0)
- added J66: Conn_02x01, Wire_Connections_Bridges:WireConnection_1.00mmDrill, F.Cu at (109.2, 260.0)
- added J67: Conn_02x01, Wire_Connections_Bridges:WireConnection_1.00mmDrill, F.Cu at (194.0, 226.8)
- added J68: Screw_Terminal_01x02, Connectors_Terminal_Blocks:TerminalBlock_bornier-2_P5.08mm, F.Cu at (193.9, 246.0)
- added J69: Conn_02x01, Wire_Connections_Bridges:WireConnection_1.00mmDrill, F.Cu at (199.0, 226.8)
- added R1: 10k, Wire_Connections_Bridges:WireConnection_1.00mmDrill, F.Cu at (224.0, 55.8)
- added R2: 2k7, Wire_Connections_Bridges:WireConnection_1.00mmDrill, F.Cu at (224.0, 71.8)
- added REF**: MountingHole_4.3mm_M4, Mounting_Holes:MountingHole_4.3mm_M4, F.Cu at (168.0, 172.0)
- added REF**: MountingHole_4.3mm_M4, Mounting_Holes:MountingHole_4.3mm_M4, F.Cu at (168.0, 32.0)
- added REF**: MountingHole_4.3mm_M4, Mounting_Holes:MountingHole_4.3mm_M4, F.Cu at (28.0, 172.0)
- added REF**: MountingHole_4.3mm_M4, Mounting_Holes:MountingHole_4.3mm_M4, F.Cu at (28.0, 32.0)
- J1: value I2S_DAC -> Conn_02x01; footprint Socket_Strips:Socket_Strip_Straight_1x06_Pitch2.54mm -> Wire_Connections_Bridges:WireConnection_1.00mmDrill
- J10, J12, J13, J14, J5, J6, J7, J8, J9: value Conn_01x06_Male -> Conn_02x01; footprint Moederbord:IDC_Header_Straight_6pins -> Wire_Connections_Bridges:WireConnection_1.00mmDrill
- J11: value Conn_01x06_Male -> Conn_01x06_Female
- J15, J16: value Conn_01x06_Male -> Conn_01x12_Female; footprint Moederbord:IDC_Header_Straight_6pins -> Socket_Strips:Socket_Strip_Straight_1x12_Pitch2.54mm
- J17: value Conn_01x06_Male -> Screw_Terminal_01x02; footprint Moederbord:IDC_Header_Straight_6pins -> Connectors_Terminal_Blocks:TerminalBlock_bornier-2_P5.08mm
- J2: value RFID_reader -> Conn_02x01; footprint Socket_Strips:Socket_Strip_Straight_1x08_Pitch2.54mm -> Wire_Connections_Bridges:WireConnection_1.00mmDrill
- J3: value ESP32_left -> Conn_02x01; footprint Socket_Strips:Socket_Strip_Straight_1x15_Pitch2.54mm -> Wire_Connections_Bridges:WireConnection_1.00mmDrill
- J4: value ESP32_right -> I2S_DAC; footprint Socket_Strips:Socket_Strip_Straight_1x15_Pitch2.54mm -> Socket_Strips:Socket_Strip_Straight_1x06_Pitch2.54mm
- moved J5 216.0 mm to (-21.2, 51.0)
- moved J1 196.4 mm to (-21.2, 42.0), turned to 0 degrees
- moved J2 149.3 mm to (-21.2, 45.0), turned to 0 degrees
- moved J17 138.1 mm to (224.0, 47.0)
- moved J27 133.6 mm to (29.6, 100.5)
- moved J6 128.3 mm to (-21.2, 54.0)
- moved J28 119.3 mm to (48.3, 100.5)
- moved J4 113.4 mm to (-6.00, 43.4)
- moved J7 109.9 mm to (-21.2, 57.0)
- moved J29 107.6 mm to (67.1, 100.5)
- moved J3 106.3 mm to (-21.2, 48.0)
- moved J14 105.7 mm to (71.2, 134.0), turned to 180 degrees
- moved U2 105.6 mm to (83.7, 230.5)
- moved U1 105.6 mm to (84.0, 207.0)
- moved U3 105.6 mm to (83.4, 254.5)
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Connections:
- J1 pad 1: (no net) -> DAC_BCK
- J1 pad 2: (no net) -> Net-(J1-Pad2)
- J10 pad 1: +5V -> RFID_MOSI
- J11 pad 1: +5V -> Net-(J11-Pad1)
- J11 pad 2: Net-(J10-Pad3) -> Net-(J11-Pad2)
- J11 pad 3: Net-(J11-Pad3) -> Net-(J10-Pad2)
- J11 pad 4: (no net) -> Net-(J11-Pad4)
- J11 pad 5: GND -> Net-(J11-Pad5)
- J11 pad 6: (no net) -> Net-(J11-Pad6)
- J12 pad 1: +5V -> RFID_MISO
- J12 pad 2: Net-(J11-Pad3) -> Net-(J11-Pad4)
- J13 pad 1: +5V -> GND
- J13 pad 2: Net-(J12-Pad3) -> Net-(J11-Pad5)
- J14 pad 1: +5V -> +3V3
- J14 pad 2: Net-(J13-Pad3) -> Net-(J11-Pad6)
- J15 pad 1: +5V -> GND
- J15 pad 2: Net-(J14-Pad3) -> GND
- J15 pad 3: Net-(J15-Pad3) -> Shift_CLK
- J15 pad 4: (no net) -> Shift_SH_LDn1
- J15 pad 5: GND -> Shift_SH_LDn2
- J15 pad 6: (no net) -> Shift_SH_LDn3
- J16 pad 1: +5V -> +3V3
- J16 pad 2: Net-(J15-Pad3) -> Shift_data
- J16 pad 3: Net-(J16-Pad3) -> Touch_menu
- J16 pad 4: (no net) -> RFID_MISO
- J16 pad 5: GND -> BatMon
- J16 pad 6: (no net) -> DAC_DATA
- J17 pad 1: +5V -> Net-(J17-Pad1)
- J17 pad 2: Net-(J16-Pad3) -> (no net)
- J18 pad 2: Net-(J17-Pad3) -> LED_rings_data
- J18 pad 4: (no net) -> Touch_menu
- J19 pad 4: (no net) -> Touch1
- J2 pad 1: (no net) -> DAC_DATA
- J2 pad 2: (no net) -> Net-(J2-Pad2)
- J20 pad 4: (no net) -> Touch2
- J21 pad 4: (no net) -> Touch3
- J22 pad 4: (no net) -> Touch4
- J23 pad 4: (no net) -> Touch5
- J24 pad 4: (no net) -> Touch6
- J25 pad 4: (no net) -> Touch7
- J26 pad 4: (no net) -> Touch8
- J27 pad 4: (no net) -> Touch9
- J28 pad 4: (no net) -> Touch10
- J29 pad 3: (no net) -> Net-(J29-Pad3)
- J29 pad 4: (no net) -> Touch11
- J3 pad 1: (no net) -> DAC_LRCK
- J3 pad 2: (no net) -> Net-(J3-Pad2)
- J4 pad 1: (no net) -> Net-(J1-Pad2)
- J4 pad 2: (no net) -> Net-(J2-Pad2)
- J4 pad 3: (no net) -> Net-(J3-Pad2)
- J4 pad 4: (no net) -> Net-(J4-Pad4)
- J4 pad 5: (no net) -> Net-(J4-Pad5)
- J4 pad 6: (no net) -> Net-(J4-Pad6)
- J5 pad 1: +5V -> GND
- J5 pad 2: (no net) -> Net-(J4-Pad4)
- J6 pad 1: +5V -> GND
- J6 pad 2: Net-(J5-Pad3) -> Net-(J4-Pad5)
- J7 pad 1: +5V -> +3V3
- J7 pad 2: Net-(J6-Pad3) -> Net-(J4-Pad6)
- J8 pad 1: +5V -> RFID_CS
- J8 pad 2: Net-(J7-Pad3) -> Net-(J11-Pad1)
- J9 pad 1: +5V -> RFID_SCLK
- J9 pad 2: Net-(J8-Pad3) -> Net-(J11-Pad2)
- U1 pad 1: (no net) -> GND
- U1 pad 10: (no net) -> Net-(J47-Pad2)
- U1 pad 11: (no net) -> Net-(J48-Pad2)
- U1 pad 12: (no net) -> Net-(J49-Pad2)
- U1 pad 14: (no net) -> Net-(J50-Pad2)
- U1 pad 15: (no net) -> Shift_SH_LDn1
- U1 pad 2: (no net) -> Net-(J43-Pad2)
- U1 pad 3: (no net) -> Net-(J44-Pad2)
- U1 pad 4: (no net) -> Net-(J45-Pad2)
- U1 pad 5: (no net) -> Net-(J46-Pad2)
- U1 pad 6: (no net) -> GND
- U1 pad 7: (no net) -> Shift_CLK
- U1 pad 9: (no net) -> +3V3
- U2 pad 10: (no net) -> Net-(J55-Pad2)
- U2 pad 11: (no net) -> Net-(J56-Pad2)
- U2 pad 12: (no net) -> Net-(J57-Pad2)
- U2 pad 14: (no net) -> Net-(J58-Pad2)
- U2 pad 15: (no net) -> Shift_SH_LDn2
- U2 pad 2: (no net) -> Net-(J51-Pad2)
- U2 pad 3: (no net) -> Net-(J52-Pad2)
- U2 pad 4: (no net) -> Net-(J53-Pad2)
- U2 pad 5: (no net) -> Net-(J54-Pad2)
- U2 pad 6: (no net) -> GND
- U2 pad 7: (no net) -> Shift_CLK
- U2 pad 9: (no net) -> +3V3
- U3 pad 10: (no net) -> Net-(J63-Pad2)
- U3 pad 11: (no net) -> Net-(J64-Pad2)
- U3 pad 12: (no net) -> Net-(J65-Pad2)
- U3 pad 13: (no net) -> Shift_data
- U3 pad 14: (no net) -> Net-(J66-Pad2)
- U3 pad 15: (no net) -> Shift_SH_LDn3
- U3 pad 2: (no net) -> Net-(J59-Pad2)
- U3 pad 3: (no net) -> Net-(J60-Pad2)
- U3 pad 4: (no net) -> Net-(J61-Pad2)
- U3 pad 5: (no net) -> Net-(J62-Pad2)
- U3 pad 6: (no net) -> GND
- U3 pad 7: (no net) -> Shift_CLK
- U3 pad 9: (no net) -> +3V3

Commit message: Update moederbord
Parts:
- removed J1, J10, J12, J13, J14, J2, J3, J43, J44, J45, J46, J47, J48, J49, J5, J50, J51, J52, J53, J54, J55, J56, J57, J58, J59, J6, J60, J61, J62, J63, J64, J65, J66, J67, J69, J7, J8, J9: Conn_02x01, Wire_Connections_Bridges:WireConnection_1.00mmDrill
- added JP1: Jumper, Moederbord:Jumper_1x2_Pitch2.54mm, F.Cu at (70.0, 128.0)
- added JP10: Jumper, Moederbord:Jumper_1x2_Pitch2.54mm, F.Cu at (39.0, 129.0)
- added JP11: Jumper, Moederbord:Jumper_1x2_Pitch2.54mm, F.Cu at (132.0, 131.0)
- added JP12: Jumper, Moederbord:Jumper_1x2_Pitch2.54mm, F.Cu at (39.0, 134.0)
- added JP13: Jumper, Moederbord:Jumper_1x2_Pitch2.54mm, F.Cu at (132.0, 134.0)
- added JP14: Jumper, Moederbord:Jumper_1x2_Pitch2.54mm, F.Cu at (132.0, 137.0)
- added JP15: Jumper, Moederbord:Jumper_1x2_Pitch2.54mm, F.Cu at (41.0, 67.0)
- added JP16: Jumper, Moederbord:Jumper_1x2_Pitch2.54mm, F.Cu at (41.0, 70.0)
- added JP17: Jumper, Moederbord:Jumper_1x2_Pitch2.54mm, F.Cu at (41.0, 73.0)
- added JP18: Jumper, Moederbord:Jumper_1x2_Pitch2.54mm, F.Cu at (41.0, 76.0)
- added JP19: Jumper, Moederbord:Jumper_1x2_Pitch2.54mm, F.Cu at (65.0, 81.0)
- added JP2: Jumper, Moederbord:Jumper_1x2_Pitch2.54mm, F.Cu at (93.0, 128.0)
- added JP20: Jumper, Moederbord:Jumper_1x2_Pitch2.54mm, F.Cu at (65.0, 78.0)
- added JP21: Jumper, Moederbord:Jumper_1x2_Pitch2.54mm, F.Cu at (65.0, 75.0)
- added JP22: Jumper, Moederbord:Jumper_1x2_Pitch2.54mm, F.Cu at (65.0, 70.0)
- added JP23: Jumper, Moederbord:Jumper_1x2_Pitch2.54mm, F.Cu at (72.0, 65.0)
- added JP24: Jumper, Moederbord:Jumper_1x2_Pitch2.54mm, F.Cu at (72.0, 68.0)
- added JP25: Jumper, Moederbord:Jumper_1x2_Pitch2.54mm, F.Cu at (72.0, 71.0)
- added JP26: Jumper, Moederbord:Jumper_1x2_Pitch2.54mm, F.Cu at (72.0, 74.0)
- added JP27: Jumper, Moederbord:Jumper_1x2_Pitch2.54mm, F.Cu at (96.0, 79.0)
- added JP28: Jumper, Moederbord:Jumper_1x2_Pitch2.54mm, F.Cu at (96.0, 76.0)
- added JP29: Jumper, Moederbord:Jumper_1x2_Pitch2.54mm, F.Cu at (96.0, 73.0)
- added JP3: Jumper, Moederbord:Jumper_1x2_Pitch2.54mm, F.Cu at (70.0, 131.0)
- added JP30: Jumper, Moederbord:Jumper_1x2_Pitch2.54mm, F.Cu at (96.0, 68.0)
- added JP31: Jumper, Moederbord:Jumper_1x2_Pitch2.54mm, F.Cu at (104.0, 65.0)
- added JP32: Jumper, Moederbord:Jumper_1x2_Pitch2.54mm, F.Cu at (104.0, 68.0)
- added JP33: Jumper, Moederbord:Jumper_1x2_Pitch2.54mm, F.Cu at (104.0, 71.0)
- added JP34: Jumper, Moederbord:Jumper_1x2_Pitch2.54mm, F.Cu at (104.0, 74.0)
- added JP35: Jumper, Moederbord:Jumper_1x2_Pitch2.54mm, F.Cu at (128.0, 79.0)
- added JP36: Jumper, Moederbord:Jumper_1x2_Pitch2.54mm, F.Cu at (128.0, 76.0)
- added JP37: Jumper, Moederbord:Jumper_1x2_Pitch2.54mm, F.Cu at (128.0, 73.0)
- added JP38: Jumper, Moederbord:Jumper_1x2_Pitch2.54mm, F.Cu at (128.0, 68.0)
- added JP4: Jumper, Moederbord:Jumper_1x2_Pitch2.54mm, F.Cu at (93.0, 131.0)
- added JP5: Jumper, Moederbord:Jumper_1x2_Pitch2.54mm, F.Cu at (70.0, 134.0)
- added JP6: Jumper, Moederbord:Jumper_1x2_Pitch2.54mm, F.Cu at (93.0, 134.0)
- added JP7: Jumper, Moederbord:Jumper_1x2_Pitch2.54mm, F.Cu at (132.0, 122.0)
- added JP8: Jumper, Moederbord:Jumper_1x2_Pitch2.54mm, F.Cu at (132.0, 125.0)
- added JP9: Jumper, Moederbord:Jumper_1x2_Pitch2.54mm, F.Cu at (132.0, 128.0)
- J17, J68: footprint Connectors_Terminal_Blocks:TerminalBlock_bornier-2_P5.08mm -> Moederbord:TerminalBlock_2_P5.08mm
- moved J68 202.3 mm to (29.0, 128.9), turned to 270 degrees
- moved U3 193.0 mm to (111.4, 63.5)
- moved U2 167.0 mm to (79.7, 63.5)
- moved J4 166.5 mm to (140.0, 123.4)
- moved U1 146.3 mm to (48.7, 65.0)
- moved J18 117.2 mm to (29.0, 70.0), turned to 270 degrees
- moved J17 102.3 mm to (167.0, 132.0), turned to 90 degrees
- moved R1 92.2 mm to (154.0, 115.8)
- moved R2 92.2 mm to (154.0, 131.8)
- moved J11 30.0 mm to (81.0, 128.0)
Routing:
- net Net-(J18-Pad3): track 0.00 -> 30.8 mm
- net Net-(J25-Pad3): track 0.00 -> 17.4 mm
- net Net-(J33-Pad3): track 0.00 -> 17.4 mm
- net Net-(J24-Pad3): track 0.00 -> 17.2 mm
- net Net-(J22-Pad3): track 0.00 -> 17.2 mm
- net Net-(J21-Pad3): track 0.00 -> 17.2 mm
- net Net-(J20-Pad3): track 0.00 -> 17.2 mm
- net Net-(J19-Pad3): track 0.00 -> 17.2 mm
- net Net-(J23-Pad3): track 0.00 -> 17.2 mm
- net Net-(J32-Pad3): track 0.00 -> 17.2 mm
- net Net-(J30-Pad3): track 0.00 -> 17.2 mm
- net Net-(J27-Pad3): track 0.00 -> 17.2 mm
- net Net-(J29-Pad3): track 0.00 -> 17.2 mm
- net Net-(J28-Pad3): track 0.00 -> 17.2 mm
- net Net-(J31-Pad3): track 0.00 -> 17.2 mm
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