File: Elektronica/KiCad projecten/Toetsmodule/Toetsmodule.kicad_pcb (KiCad board)
At the start: 2 copper layers, 60 x 60 mm, 8 parts, among them J1 Conn_01x03_Male, J2 Touch module, J3 Conn_01x06_Male, J4 Conn_01x03_Male

Commit message: Toetsmodule v1 klaar
Parts:
- removed the J3 at (122.5, 136.5)
- removed J4: Conn_01x03_Male, Pin_Headers:Pin_Header_Straight_1x03_Pitch2.54mm
- added J2: Conn_01x06_Male, Toetsmodule:IDC_Header_Straight_6pins, B.Cu at (122.5, 138.0)
- added REF**: MountingHole_2.2mm_M2, Mounting_Holes:MountingHole_2.2mm_M2, F.Cu at (141.5, 131.5)
- added REF**: MountingHole_2.2mm_M2, Mounting_Holes:MountingHole_2.2mm_M2, F.Cu at (108.5, 131.5)
- added REF**: MountingHole_2.2mm_M2, Mounting_Holes:MountingHole_2.2mm_M2, F.Cu at (141.5, 98.5)
- added REF**: MountingHole_2.2mm_M2, Mounting_Holes:MountingHole_2.2mm_M2, F.Cu at (108.5, 98.5)
- J1: value Conn_01x03_Male -> Conn_01x04_Male; footprint Pin_Headers:Pin_Header_Straight_1x03_Pitch2.54mm -> Pin_Headers:Pin_Header_Straight_1x04_Pitch2.54mm
- moved J1 43.5 mm to (147.0, 111.0)
- renumbered J2 to J3
Connections:
- J1 pad 1: +5V -> /LED_out
- J1 pad 2: /LED_in -> GND
- J1 pad 3: GND -> +5V
- J3 pad 3: +5V -> +3V3
Routing:
- net /Touch_output: track 66.9 -> 32.1 mm
- net /LED_out: track 30.4 -> 37.1 mm
- net /LED_in: track 32.1 -> 27.4 mm
- added copper zone on F.Cu, net +3V3
Other:
- board text added: "DO GND 5V DI"
- board text added: "LEDin | 5Vin | LEDout GND | 3V3in | TOUCHout"
- board text removed: "5V Din GND"
- board text removed: "5V Dout GND"
- board text removed: "GND | LEDout | 5V NC | TOUCHout | LEDin"
