File: Elektronica/KiCad projecten/Moederbord/Moederbord.kicad_pcb (KiCad board)
At the start: 2 copper layers, 150 x 150 mm, 78 parts, among them J11 Conn_01x06_Female, J15 Conn_01x12_Female, J16 Conn_01x12_Female, J17 Screw_Terminal_01x02, J18 Conn_01x06_Male, J19 Conn_01x06_Male, J20 Conn_01x06_Male, J21 Conn_01x06_Male, J22 Conn_01x06_Male, J23 Conn_01x06_Male, J24 Conn_01x06_Male, J25 Conn_01x06_Male, J26 Conn_01x06_Male, J27 Conn_01x06_Male, J28 Conn_01x06_Male, J29 Conn_01x06_Male, J30 Conn_01x06_Male, J31 Conn_01x06_Male, J32 Conn_01x06_Male, J33 Conn_01x06_Male, J34 Conn_01x06_Male, J35 Conn_01x06_Male, J36 Conn_01x06_Male, J37 Conn_01x06_Male, J38 Conn_01x06_Male, J39 Conn_01x06_Male, J4 I2S_DAC, J40 Conn_01x06_Male, J41 Conn_01x06_Male, J42 Conn_01x06_Male, J68 Screw_Terminal_01x02, U1 74166, U2 74166, U3 74166

Commit message: Update
Parts:
- removed J38, J39, J40, J41, J42: Conn_01x06_Male, Moederbord:IDC_Header_Straight_6pins
- removed J68: Screw_Terminal_01x02, Moederbord:TerminalBlock_2_P5.08mm
- removed JP1, JP10, JP11, JP12, JP13, JP14, JP15, JP16, JP17, JP18, JP19, JP2, JP20, JP21, JP22, JP23, JP24, JP25, JP26, JP27, JP28, JP29, JP3, JP30, JP31, JP32, JP33, JP34, JP35, JP36, JP37, JP38, JP4, JP5, JP6, JP7, JP8, JP9: Jumper, Moederbord:Jumper_1x2_Pitch2.54mm
- added C1: 100 uF, Capacitors_SMD:C_1210_HandSoldering, F.Cu at (42.0, 131.0)
- added C2: 100 uF, Capacitors_SMD:C_1210_HandSoldering, F.Cu at (87.0, 128.0)
- added C3: 100 uF, Capacitors_SMD:C_1210_HandSoldering, F.Cu at (87.0, 133.0)
- added C4: 100 uF, Capacitors_SMD:C_1210_HandSoldering, F.Cu at (62.0, 61.0)
- added C5: 100 uF, Capacitors_SMD:C_1210_HandSoldering, F.Cu at (97.0, 61.0)
- added C6: 100 uF, Capacitors_SMD:C_1210_HandSoldering, F.Cu at (132.0, 61.0)
- added J1: Conn_02x06_Top_Bottom, Pin_Headers:Pin_Header_Straight_2x06_Pitch2.54mm, F.Cu at (111.5, 127.5)
- added J10: Conn_01x06_Male, Moederbord:IDC_Header_Straight_6pins, F.Cu at (29.0, 70.0)
- added J12: Conn_01x06_Male, Moederbord:IDC_Header_Straight_6pins, F.Cu at (48.7, 44.7)
- added J13: Conn_01x06_Male, Moederbord:IDC_Header_Straight_6pins, F.Cu at (67.4, 44.7)
- added J14: Conn_01x06_Male, Moederbord:IDC_Header_Straight_6pins, F.Cu at (86.1, 44.7)
- added J2: I2S_DAC, Socket_Strips:Socket_Strip_Straight_1x06_Pitch2.54mm, F.Cu at (121.0, 127.5)
- added J3: Conn_02x02_Top_Bottom, Pin_Headers:Pin_Header_Straight_2x02_Pitch2.54mm, F.Cu at (37.0, 130.0)
- added J5: Conn_02x06_Top_Bottom, Pin_Headers:Pin_Header_Straight_2x06_Pitch2.54mm, F.Cu at (157.0, 80.0)
- added J6: Conn_01x06_Female, Moederbord:IDC_Header_Straight_6pins, F.Cu at (168.0, 76.0)
- added J7: Conn_01x12_Female, Socket_Strips:Socket_Strip_Straight_1x12_Pitch2.54mm, F.Cu at (60.0, 124.0)
- added J8: Conn_01x12_Female, Socket_Strips:Socket_Strip_Straight_1x12_Pitch2.54mm, F.Cu at (60.0, 137.0)
- added J9: Screw_Terminal_01x02, Moederbord:TerminalBlock_2_P5.08mm, F.Cu at (167.0, 125.1)
- J11: value Conn_01x06_Female -> Conn_01x06_Male
- J15, J16: value Conn_01x12_Female -> Conn_01x06_Male; footprint Socket_Strips:Socket_Strip_Straight_1x12_Pitch2.54mm -> Moederbord:IDC_Header_Straight_6pins
- J17: value Screw_Terminal_01x02 -> Conn_01x06_Male; footprint Moederbord:TerminalBlock_2_P5.08mm -> Moederbord:IDC_Header_Straight_6pins
- J35, J36, J37: value Conn_01x06_Male -> Conn_02x08_Odd_Even; footprint Moederbord:IDC_Header_Straight_6pins -> Pin_Headers:Pin_Header_Straight_2x08_Pitch2.54mm
- J4: value I2S_DAC -> Screw_Terminal_01x02; footprint Socket_Strips:Socket_Strip_Straight_1x06_Pitch2.54mm -> Moederbord:TerminalBlock_2_P5.08mm
- moved J18 134.4 mm to (161.0, 44.5), turned to 0 degrees
- moved J4 112.1 mm to (28.0, 129.0), turned to 270 degrees
- moved J37 105.7 mm to (116.5, 65.5)
- moved J36 99.5 mm to (82.5, 65.5)
- moved J11 97.7 mm to (30.0, 44.7), turned to 0 degrees
- moved J35 95.1 mm to (47.0, 65.5)
- moved J17 90.9 mm to (142.3, 44.5), turned to 0 degrees
- moved J27 61.0 mm to (29.6, 161.5)
- moved J28 61.0 mm to (48.3, 161.5)
- moved J29 61.0 mm to (67.1, 161.5)
- moved J30 61.0 mm to (85.8, 161.5)
- moved J31 61.0 mm to (104.5, 161.5)
- moved J32 61.0 mm to (123.2, 161.5)
- moved J33 61.0 mm to (141.9, 161.5)
- moved J34 60.5 mm to (161.0, 161.5)
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Connections:
- J11 pad 2: Net-(J11-Pad2) -> Touch1
- J11 pad 3: Net-(J11-Pad3) -> +5V
- J11 pad 4: Net-(J11-Pad4) -> +3V3
- J11 pad 6: Net-(J11-Pad6) -> GND
- J15 pad 1: GND -> Net-(J15-Pad1)
- J15 pad 2: GND -> Touch5
- J15 pad 3: Shift_CLK -> +5V
- J15 pad 4: Shift_SH_LDn1 -> +3V3
- J15 pad 5: Shift_SH_LDn2 -> Net-(J14-Pad1)
- J15 pad 6: Shift_SH_LDn3 -> GND
- J16 pad 1: +3V3 -> Net-(J16-Pad1)
- J16 pad 2: Shift_data -> Touch6
- J16 pad 3: Touch_menu -> +5V
- J16 pad 4: RFID_MISO -> +3V3
- J16 pad 5: BatMon -> Net-(J15-Pad1)
- J16 pad 6: DAC_DATA -> GND
- J17 pad 2: (no net) -> Touch7
- J18 pad 1: +5V -> Net-(J18-Pad1)
- J18 pad 2: LED_rings_data -> Touch8
- J18 pad 3: Net-(J18-Pad3) -> +5V
- J18 pad 4: Touch_menu -> +3V3
- J18 pad 5: GND -> Net-(J17-Pad1)
- J18 pad 6: (no net) -> GND
- J19 pad 1: +5V -> Net-(J19-Pad1)
- J19 pad 2: Net-(J18-Pad3) -> Touch9
- J19 pad 3: Net-(J19-Pad3) -> +5V
- J19 pad 4: Touch1 -> +3V3
- J19 pad 5: GND -> Net-(J18-Pad1)
- J19 pad 6: (no net) -> GND
- J20 pad 1: +5V -> Net-(J20-Pad1)
- J20 pad 2: Net-(J19-Pad3) -> Touch10
- J20 pad 3: Net-(J20-Pad3) -> +5V
- J20 pad 4: Touch2 -> +3V3
- J20 pad 5: GND -> Net-(J19-Pad1)
- J20 pad 6: (no net) -> GND
- J21 pad 1: +5V -> Net-(J21-Pad1)
- J21 pad 2: Net-(J20-Pad3) -> Touch11
- J21 pad 3: Net-(J21-Pad3) -> +5V
- J21 pad 4: Touch3 -> +3V3
- J21 pad 5: GND -> Net-(J20-Pad1)
- J21 pad 6: (no net) -> GND
- J22 pad 1: +5V -> Net-(J22-Pad1)
- J22 pad 2: Net-(J21-Pad3) -> Touch12
- J22 pad 3: Net-(J22-Pad3) -> +5V
- J22 pad 4: Touch4 -> +3V3
- J22 pad 5: GND -> Net-(J21-Pad1)
- J22 pad 6: (no net) -> GND
- J23 pad 1: +5V -> Net-(J23-Pad1)
- J23 pad 2: Net-(J22-Pad3) -> Touch13
- J23 pad 3: Net-(J23-Pad3) -> +5V
- J23 pad 4: Touch5 -> +3V3
- J23 pad 5: GND -> Net-(J22-Pad1)
- J23 pad 6: (no net) -> GND
- J24 pad 1: +5V -> Net-(J24-Pad1)
- J24 pad 2: Net-(J23-Pad3) -> Touch14
- J24 pad 3: Net-(J24-Pad3) -> +5V
- J24 pad 4: Touch6 -> +3V3
- J24 pad 5: GND -> Net-(J23-Pad1)
- J24 pad 6: (no net) -> GND
- J25 pad 1: +5V -> Net-(J25-Pad1)
- J25 pad 2: Net-(J24-Pad3) -> Touch15
- J25 pad 3: Net-(J25-Pad3) -> +5V
- J25 pad 4: Touch7 -> +3V3
- J25 pad 5: GND -> Net-(J24-Pad1)
- J25 pad 6: (no net) -> GND
- J26 pad 1: +5V -> Net-(J26-Pad1)
- J26 pad 2: Net-(J25-Pad3) -> Touch16
- J26 pad 3: Net-(J26-Pad3) -> +5V
- J26 pad 4: Touch8 -> +3V3
- J26 pad 5: GND -> Net-(J25-Pad1)
- J26 pad 6: (no net) -> GND
- J27 pad 1: +5V -> Net-(J27-Pad1)
- J27 pad 2: Net-(J26-Pad3) -> Touch17
- J27 pad 3: Net-(J27-Pad3) -> +5V
- J27 pad 4: Touch9 -> +3V3
- J27 pad 5: GND -> Net-(J26-Pad1)
- J27 pad 6: (no net) -> GND
- J28 pad 1: +5V -> Net-(J28-Pad1)
- J28 pad 2: Net-(J27-Pad3) -> Touch18
- J28 pad 3: Net-(J28-Pad3) -> +5V
- J28 pad 4: Touch10 -> +3V3
- J28 pad 5: GND -> Net-(J27-Pad1)
- J28 pad 6: (no net) -> GND
- J29 pad 1: +5V -> Net-(J29-Pad1)
- J29 pad 2: Net-(J28-Pad3) -> Touch19
- J29 pad 3: Net-(J29-Pad3) -> +5V
- J29 pad 4: Touch11 -> +3V3
- J29 pad 5: GND -> Net-(J28-Pad1)
- J29 pad 6: (no net) -> GND
- J30 pad 1: +5V -> Net-(J30-Pad1)
- J30 pad 2: Net-(J29-Pad3) -> Touch20
- J30 pad 3: Net-(J30-Pad3) -> +5V
- J30 pad 4: Touch12 -> +3V3
- J30 pad 5: GND -> Net-(J29-Pad1)
- J30 pad 6: (no net) -> GND
- J31 pad 1: +5V -> Net-(J31-Pad1)
- J31 pad 2: Net-(J30-Pad3) -> Touch21
- J31 pad 3: Net-(J31-Pad3) -> +5V
- J31 pad 4: Touch13 -> +3V3
- J31 pad 5: GND -> Net-(J30-Pad1)
- J31 pad 6: (no net) -> GND
- J32 pad 1: +5V -> Net-(J32-Pad1)
- J32 pad 2: Net-(J31-Pad3) -> Touch22
- J32 pad 3: Net-(J32-Pad3) -> +5V
- J32 pad 4: Touch14 -> +3V3
- J32 pad 5: GND -> Net-(J31-Pad1)
- J32 pad 6: (no net) -> GND
- J33 pad 1: +5V -> Net-(J33-Pad1)
- J33 pad 2: Net-(J32-Pad3) -> Touch23
- J33 pad 3: Net-(J33-Pad3) -> +5V
- J33 pad 4: Touch15 -> +3V3
- J33 pad 5: GND -> Net-(J32-Pad1)
- J33 pad 6: (no net) -> GND
- J34 pad 1: +5V -> (no net)
- J34 pad 2: Net-(J33-Pad3) -> Touch24
- J34 pad 3: Net-(J34-Pad3) -> +5V
- J34 pad 4: Touch16 -> +3V3
- J34 pad 5: GND -> Net-(J33-Pad1)
- J34 pad 6: (no net) -> GND
- J35 pad 1: +5V -> Touch1
- J35 pad 2: Net-(J34-Pad3) -> Net-(J35-Pad2)
- J35 pad 3: Net-(J35-Pad3) -> Touch2
- J35 pad 4: Touch17 -> Net-(J35-Pad4)
- J35 pad 5: GND -> Touch3
- J35 pad 6: (no net) -> Net-(J35-Pad6)
- J36 pad 1: +5V -> Touch9
- J36 pad 2: Net-(J35-Pad3) -> Net-(J36-Pad2)
- J36 pad 3: Net-(J36-Pad3) -> Touch10
- J36 pad 4: Touch18 -> Net-(J36-Pad4)
- J36 pad 5: GND -> Touch11
- J36 pad 6: (no net) -> Net-(J36-Pad6)
- J37 pad 1: +5V -> Touch17
- J37 pad 2: Net-(J36-Pad3) -> Net-(J37-Pad2)
- J37 pad 3: Net-(J37-Pad3) -> Touch18
- J37 pad 4: Touch19 -> Net-(J37-Pad4)
- J37 pad 5: GND -> Touch19
- J37 pad 6: (no net) -> Net-(J37-Pad6)
- R1 pad 1: Net-(J17-Pad1) -> Net-(J9-Pad1)
- U1 pad 10: Net-(JP19-Pad2) -> Net-(J35-Pad10)
- U1 pad 11: Net-(JP20-Pad2) -> Net-(J35-Pad12)
- U1 pad 12: Net-(JP21-Pad2) -> Net-(J35-Pad14)
- U1 pad 14: Net-(JP22-Pad2) -> Net-(J35-Pad16)
- U1 pad 16: VCC -> +3V3
- U1 pad 2: Net-(JP15-Pad2) -> Net-(J35-Pad2)
- U1 pad 3: Net-(JP16-Pad2) -> Net-(J35-Pad4)
- U1 pad 4: Net-(JP17-Pad2) -> Net-(J35-Pad6)
- U1 pad 5: Net-(JP18-Pad2) -> Net-(J35-Pad8)
- U2 pad 10: Net-(JP27-Pad2) -> Net-(J36-Pad10)
- U2 pad 11: Net-(JP28-Pad2) -> Net-(J36-Pad12)
- U2 pad 12: Net-(JP29-Pad2) -> Net-(J36-Pad14)
- U2 pad 14: Net-(JP30-Pad2) -> Net-(J36-Pad16)
- U2 pad 16: VCC -> +3V3
- U2 pad 2: Net-(JP23-Pad2) -> Net-(J36-Pad2)
- U2 pad 3: Net-(JP24-Pad2) -> Net-(J36-Pad4)
- U2 pad 4: Net-(JP25-Pad2) -> Net-(J36-Pad6)
- U2 pad 5: Net-(JP26-Pad2) -> Net-(J36-Pad8)
- U3 pad 10: Net-(JP35-Pad2) -> Net-(J37-Pad10)
- U3 pad 11: Net-(JP36-Pad2) -> Net-(J37-Pad12)
- U3 pad 12: Net-(JP37-Pad2) -> Net-(J37-Pad14)
- U3 pad 14: Net-(JP38-Pad2) -> Net-(J37-Pad16)
- U3 pad 16: VCC -> +3V3
- U3 pad 2: Net-(JP31-Pad2) -> Net-(J37-Pad2)
- U3 pad 3: Net-(JP32-Pad2) -> Net-(J37-Pad4)
- U3 pad 4: Net-(JP33-Pad2) -> Net-(J37-Pad6)
- U3 pad 5: Net-(JP34-Pad2) -> Net-(J37-Pad8)
Routing:
- net GND: track 0.00 -> 67.5 mm
- net Net-(J18-Pad3): track 30.8 -> 0.00 mm
- net +3V3: track 0.00 -> 19.8 mm
- net Net-(J25-Pad3): track 17.4 -> 0.00 mm
- net Net-(J33-Pad3): track 17.4 -> 0.00 mm
- net Net-(J24-Pad3): track 17.2 -> 0.00 mm
- net Net-(J22-Pad3): track 17.2 -> 0.00 mm
- net Net-(J21-Pad3): track 17.2 -> 0.00 mm
- net Net-(J20-Pad3): track 17.2 -> 0.00 mm
- net Net-(J19-Pad3): track 17.2 -> 0.00 mm
- net Net-(J23-Pad3): track 17.2 -> 0.00 mm
- net Net-(J32-Pad3): track 17.2 -> 0.00 mm
- net Net-(J30-Pad3): track 17.2 -> 0.00 mm
- net Net-(J27-Pad3): track 17.2 -> 0.00 mm
- net Net-(J29-Pad3): track 17.2 -> 0.00 mm
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
Commit message: Update moederbord
Parts:
- removed the J37 at (116.5, 65.5)
- added J35: Conn_02x08_Odd_Even, Pin_Headers:Pin_Header_Straight_2x08_Pitch2.54mm, F.Cu at (47.0, 65.5)
- added J38: Conn_01x03, Pin_Headers:Pin_Header_Straight_1x03_Pitch2.54mm, F.Cu at (26.9, 62.0)
- added J39: Conn_01x03, Pin_Headers:Pin_Header_Straight_1x03_Pitch2.54mm, F.Cu at (169.0, 130.0)
- added J40: Conn_02x12_Odd_Even, Pin_Headers:Pin_Header_Straight_2x12_Pitch2.54mm, F.Cu at (58.7, 109.5)
- added J41: Conn_02x12_Odd_Even, Pin_Headers:Pin_Header_Straight_2x12_Pitch2.54mm, F.Cu at (58.7, 146.0)
- J1, J5: value Conn_02x06_Top_Bottom -> Conn_02x06_Odd_Even
- moved J37 69.0 mm to (116.0, 66.0)
- moved C3 54.1 mm to (33.0, 129.0), turned to 90 degrees
- moved J3 51.0 mm to (88.0, 130.0)
- moved J4 51.0 mm to (79.0, 129.0)
- moved C1 50.0 mm to (92.0, 131.0)
- moved C2 29.0 mm to (58.0, 129.0), turned to 90 degrees
- moved R2 14.7 mm to (141.0, 125.0), turned to 180 degrees
- moved R1 10.4 mm to (159.0, 125.0), turned to 180 degrees
- moved J7 7.12 mm to (58.7, 117.0), turned to 270 degrees
- moved J5 4.00 mm to (153.0, 80.2)
- moved J8 3.27 mm to (58.7, 140.0), turned to 270 degrees
- moved J10 2.00 mm to (31.0, 70.0)
- moved J36 1.08 mm to (81.5, 65.5)
- moved J1 0.55 mm to (112.0, 127.4)
- renumbered J35 to J37
Connections:
- net Net-(J36-Pad10) renamed /Shift registers/T13
- net Net-(J36-Pad12) renamed /Shift registers/T14
- net Net-(J36-Pad14) renamed /Shift registers/T15
- net Net-(J36-Pad16) renamed /Shift registers/T16
- net Net-(J36-Pad2) renamed /Shift registers/T9
- net Net-(J36-Pad4) renamed /Shift registers/T10
- net Net-(J36-Pad6) renamed /Shift registers/T11
- net Net-(J36-Pad8) renamed /Shift registers/T12
- net Net-(U1-Pad13) renamed /Shift registers/s1_s2
- net Net-(U2-Pad13) renamed /Shift registers/s2_s3
- C2 pad 1: +3V3 -> Net-(C2-Pad1)
- C2 pad 2: GND -> Net-(C2-Pad2)
- C3 pad 1: +5V -> Net-(C3-Pad1)
- C3 pad 2: GND -> Net-(C3-Pad2)
- J1 pad 11: Net-(J1-Pad11) -> +5V
- J1 pad 2: DAC_DATA -> Net-(J1-Pad2)
- J1 pad 3: DAC_LRCK -> DAC_DATA
- J1 pad 4: GND -> Net-(J1-Pad4)
- J1 pad 5: GND -> DAC_LRCK
- J1 pad 6: +5V -> Net-(J1-Pad6)
- J1 pad 7: Net-(J1-Pad7) -> GND
- J1 pad 9: Net-(J1-Pad9) -> GND
- J2 pad 1: Net-(J1-Pad7) -> Net-(J1-Pad2)
- J2 pad 2: Net-(J1-Pad8) -> Net-(J1-Pad4)
- J2 pad 3: Net-(J1-Pad9) -> Net-(J1-Pad6)
- J2 pad 4: Net-(J1-Pad10) -> Net-(J1-Pad8)
- J2 pad 5: Net-(J1-Pad11) -> Net-(J1-Pad10)
- J37 pad 1: Touch1 -> Touch17
- J37 pad 10: Net-(J35-Pad10) -> /Shift registers/T21
- J37 pad 11: Touch6 -> Touch22
- J37 pad 12: Net-(J35-Pad12) -> /Shift registers/T22
- J37 pad 13: Touch7 -> Touch23
- J37 pad 14: Net-(J35-Pad14) -> /Shift registers/T23
- J37 pad 15: Touch8 -> Touch24
- J37 pad 16: Net-(J35-Pad16) -> /Shift registers/T24
- J37 pad 2: Net-(J35-Pad2) -> /Shift registers/T17
- J37 pad 3: Touch2 -> Touch18
- J37 pad 4: Net-(J35-Pad4) -> /Shift registers/T18
- J37 pad 5: Touch3 -> Touch19
- J37 pad 6: Net-(J35-Pad6) -> /Shift registers/T19
- J37 pad 7: Touch4 -> Touch20
- J37 pad 8: Net-(J35-Pad8) -> /Shift registers/T20
- J37 pad 9: Touch5 -> Touch21
- J5 pad 1: RFID_CS -> Net-(J5-Pad1)
- J5 pad 10: Net-(J5-Pad10) -> GND
- J5 pad 12: Net-(J5-Pad12) -> +3V3
- J5 pad 2: RFID_SCLK -> RFID_CS
- J5 pad 3: RFID_MOSI -> Net-(J5-Pad3)
- J5 pad 4: RFID_MISO -> RFID_SCLK
- J5 pad 5: GND -> Net-(J5-Pad5)
- J5 pad 6: +3V3 -> RFID_MOSI
- J5 pad 8: Net-(J5-Pad8) -> RFID_MISO
- J6 pad 1: Net-(J5-Pad7) -> Net-(J5-Pad1)
- J6 pad 2: Net-(J5-Pad8) -> Net-(J5-Pad3)
- J6 pad 3: Net-(J5-Pad9) -> Net-(J5-Pad5)
- J6 pad 4: Net-(J5-Pad10) -> Net-(J5-Pad7)
- J6 pad 5: Net-(J5-Pad11) -> Net-(J5-Pad9)
- J6 pad 6: Net-(J5-Pad12) -> Net-(J5-Pad11)
- J7 pad 1: GND -> Net-(C2-Pad2)
- J7 pad 10: GND -> Net-(J40-Pad20)
- J7 pad 11: GND -> Net-(C3-Pad2)
- J7 pad 12: +3V3 -> Net-(J40-Pad24)
- J7 pad 2: GND -> Net-(J40-Pad4)
- J7 pad 3: Shift_CLK -> Net-(J40-Pad6)
- J7 pad 4: Shift_SH_LDn1 -> Net-(J40-Pad8)
- J7 pad 5: Shift_SH_LDn2 -> Net-(J40-Pad10)
- J7 pad 6: Shift_SH_LDn3 -> Net-(J40-Pad12)
- J7 pad 7: RFID_CS -> Net-(J40-Pad14)
- J7 pad 8: RFID_MOSI -> Net-(J40-Pad16)
- J7 pad 9: RFID_SCLK -> Net-(J40-Pad18)
- J8 pad 1: +3V3 -> Net-(C2-Pad1)
- J8 pad 10: LED_display_data -> Net-(J41-Pad19)
- J8 pad 11: GND -> Net-(J41-Pad21)
- J8 pad 12: +5V -> Net-(C3-Pad1)
- J8 pad 2: Shift_data -> Net-(J41-Pad3)
- J8 pad 3: Touch_menu -> Net-(J41-Pad5)
- J8 pad 4: RFID_MISO -> Net-(J41-Pad7)
- J8 pad 5: BatMon -> Net-(J41-Pad9)
- J8 pad 6: DAC_DATA -> Net-(J41-Pad11)
- J8 pad 7: DAC_BCK -> Net-(J41-Pad13)
- J8 pad 8: DAC_LRCK -> Net-(J41-Pad15)
- J8 pad 9: LED_rings_data -> Net-(J41-Pad17)
- U1 pad 10: Net-(J35-Pad10) -> /Shift registers/T5
- U1 pad 11: Net-(J35-Pad12) -> /Shift registers/T6
- U1 pad 12: Net-(J35-Pad14) -> /Shift registers/T7
- U1 pad 14: Net-(J35-Pad16) -> /Shift registers/T8
- U1 pad 2: Net-(J35-Pad2) -> /Shift registers/T1
- U1 pad 3: Net-(J35-Pad4) -> /Shift registers/T2
- U1 pad 4: Net-(J35-Pad6) -> /Shift registers/T3
- U1 pad 5: Net-(J35-Pad8) -> /Shift registers/T4
- U3 pad 10: Net-(J37-Pad10) -> /Shift registers/T21
- U3 pad 11: Net-(J37-Pad12) -> /Shift registers/T22
- U3 pad 12: Net-(J37-Pad14) -> /Shift registers/T23
- U3 pad 14: Net-(J37-Pad16) -> /Shift registers/T24
- U3 pad 2: Net-(J37-Pad2) -> /Shift registers/T17
- U3 pad 3: Net-(J37-Pad4) -> /Shift registers/T18
- U3 pad 4: Net-(J37-Pad6) -> /Shift registers/T19
- U3 pad 5: Net-(J37-Pad8) -> /Shift registers/T20
Routing:
- net +3V3: track 19.8 -> 466.0 mm, vias 0 -> 1
- net /Shift registers/s1_s2: track 0.00 -> 31.6 mm
- net /Shift registers/s2_s3: track 0.00 -> 31.2 mm
- net Net-(J29-Pad1): track 0.00 -> 24.9 mm
- net Net-(J27-Pad1): track 0.00 -> 24.9 mm
- net Net-(J28-Pad1): track 0.00 -> 24.9 mm
- net GND: track 67.5 -> 58.2 mm
- added copper zone on B.Cu, net +3V3
- added copper zone on F.Cu, net +3V3
Other:
- board text added: "5 V in GND"
- board text added: "TTGO"
- board text added: "USB-C"

Commit message: Datasheets + update moederbord
Parts:
- moved C1 6.00 mm to (86.0, 131.0)
- moved J3 6.00 mm to (94.0, 130.0)
- moved R2 5.10 mm to (144.2, 129.0)
- moved R1 4.00 mm to (159.0, 129.0)
Connections:
- net Net-(J10-Pad1) renamed /Toetsmodules/LEDm_LED1
- net Net-(J11-Pad1) renamed /Toetsmodules/LED1_LED2
- net Net-(J12-Pad1) renamed /Toetsmodules/LED2_LED3
- net Net-(J13-Pad1) renamed /Toetsmodules/LED3_LED4
- net Net-(J14-Pad1) renamed /Toetsmodules/LED4_LED5
- net Net-(J15-Pad1) renamed /Toetsmodules/LED5_LED6
- net Net-(J16-Pad1) renamed /Toetsmodules/LED6_LED7
- net Net-(J17-Pad1) renamed /Toetsmodules/LED7_LED8
- net Net-(J18-Pad1) renamed /Toetsmodules/LED8_LED9
- net Net-(J19-Pad1) renamed /Toetsmodules/LED9_LED10
- net Net-(J20-Pad1) renamed /Toetsmodules/LED10_LED11
- net Net-(J21-Pad1) renamed /Toetsmodules/LED11_LED12
- net Net-(J22-Pad1) renamed /Toetsmodules/LED12_LED13
- net Net-(J23-Pad1) renamed /Toetsmodules/LED13_LED14
- net Net-(J24-Pad1) renamed /Toetsmodules/LED14_LED15
- net Net-(J25-Pad1) renamed /Toetsmodules/LED15_LED16
- net Net-(J26-Pad1) renamed /Toetsmodules/LED16_LED17
- net Net-(J27-Pad1) renamed /Toetsmodules/LED17_LED18
- net Net-(J28-Pad1) renamed /Toetsmodules/LED18_LED19
- net Net-(J29-Pad1) renamed /Toetsmodules/LED19_LED20
- net Net-(J30-Pad1) renamed /Toetsmodules/LED20_LED21
- net Net-(J31-Pad1) renamed /Toetsmodules/LED21_LED22
- net Net-(J32-Pad1) renamed /Toetsmodules/LED22_LED23
- net Net-(J33-Pad1) renamed /Toetsmodules/LED23_LED24
- C1 pad 1: GND -> /Conn_GND
- C1 pad 2: +5V -> /Conn_5V
- J3 pad 3: Net-(J3-Pad3) -> /Conn_5V
- J3 pad 4: Net-(J3-Pad4) -> /Conn_GND
- J4 pad 1: Net-(J3-Pad3) -> /Conn_5V
- J4 pad 2: Net-(J3-Pad4) -> /Conn_GND
Routing:
- net /Conn_GND: track 0.00 -> 13.1 mm
- net /Conn_5V: track 0.00 -> 12.9 mm
- net Net-(J3-Pad4): track 7.10 -> 0.00 mm
- net Net-(J3-Pad3): track 6.87 -> 0.00 mm
- net +5V: track 0.00 -> 2.83 mm
- net GND: track 58.2 -> 57.4 mm
Other:
- board text added: "12 V bat mon LED disp dat"
- board text added: "GND 5 V 3.3 V"
